Commit message: referencing correct lidar

File: src/ugv_description/urdf/ugv_rover.urdf (robot description, URDF)
Before this commit: robot ugv_rover, 8 links, 7 joints
Links:
- removed link base_lidar_link
- added link ldlidar_base; visual mesh filename=package://ldlidar_node/urdf/model/LD19.stl scale=0.001 0.001 0.001
- added link ldlidar_link
Joints:
- added joint ldlidar_link_joint: type fixed, parent ldlidar_base, child ldlidar_link, origin xyz=0 0 0.02745 rpy=0 0 0
- joint base_lidar_link_joint: child base_lidar_link -> ldlidar_base

Commit message: testing urdf

File: src/ugv_description/urdf/ugv_rover.urdf (robot description, URDF)
Before this commit: robot ugv_rover, 9 links, 8 joints
Joints:
- joint base_lidar_link_joint: origin xyz=0.0398145505519817 0 0.04 rpy=0 0 1.5708 -> xyz=0 0 0 rpy=0 0 0
